Commit message: Add slam_service for managing SLAM node lifecycle and update launch files
- Introduced `slam_service.py` to handle starting and stopping the SLAM node.
- Updated `CMakeLists.txt` to include `slam_service.py`.
- Modified launch files to integrate the new SLAM service and adjust parameters.
- Changed frame ID in `scan_frame_fixer.py` from 'lidar_link' to 'laser'.
- Updated URDF files to reflect changes in link names and removed unused files.

File: src/x500_description/urdf/x500_tf.urdf (robot description, URDF)
Before this commit: robot x500_tf, 3 links, 2 joints
Links:
- removed link lidar_link
- added link laser
Joints:
- joint LidarJoint: child lidar_link -> laser; origin xyz=0.1 0 0.26 rpy=0 0 0 -> xyz=0 0 0.26 rpy=0 0 0
